File: bitlight.sch (EAGLE design)
At the start: 34 parts, among them Q1 SI4126DY-T1-GE3, Q2 FDC6330L, U1 TLV521DCKT, U2 NCP500SN33, U3 MCP73833

Commit message: final design
Parts:
- removed C7: 0.1u, rcl:C-EUC0805
- removed D3: Yellow, SparkFun-LED:LED-YELLOW0603
- removed LED1: LED, rcl:C-EUC0805
- removed Q2: FDC6330L, FDC6330L:FDC6330L
- removed R10: 0.5, rcl:R-EU_R2512
- removed R11, R12, R14: 1k, rcl:R-US_R0805
- removed R13: 10k, rcl:R-US_R0805
- added P1: 3352T-1-105, 3352T-1:3352T-1
- C1, C2, C3, C4, C6: device rcl:C-EUC0805 -> rcl:C-EUC0603
- C5: value 1n -> 0.1u; device rcl:C-EUC0805 -> rcl:C-EUC0603
- D1: value RED -> 3W-AL-PCB; device SparkFun-LED:LED-RED0603 -> 3W-AL-PCB:3W-AL-PCB
- H1, H2: value MOUNT-HOLE3.0 -> MOUNT-HOLE3.6; device holes:MOUNT-HOLE3.0 -> holes:MOUNT-HOLE3.6
- R1, R2, R3: device rcl:R-US_R0805 -> rcl:R-US_R0603
- R4: value 1k -> 680; device rcl:R-US_R0805 -> rcl:R-US_R0603
- R5: value 1k -> 10k; device rcl:R-US_R0805 -> rcl:R-US_R0603
- R6: value 1k -> 7.5M; device rcl:R-US_R0805 -> rcl:R-US_R0603
- R7: value 10k -> 1k; device rcl:R-US_R0805 -> rcl:R-US_R0603
- R8: value 7.5M -> 1k; device rcl:R-US_R0805 -> rcl:R-US_R0603
- R9: value 1M-pot -> 0.5; device rcl:R-EU_R0805 -> rcl:R-EU_R2512
- U1: value TLV521DCKT -> BQ21040DBVT; device TLV521DCKT:TLV521DCKT -> BQ21040DBVT:BQ21040DBVT
- U3: value MCP73833 -> TLV521DCKT; device SparkFun-IC-Power:MCP73833 -> TLV521DCKT:TLV521DCKT
- renumbered Q1 to U4
Connections:
- removed net N$11: C2.1, Q2.VIN/R1, R13.2, U3.VBAT
- removed net N$14: C5.2, Q2.R1/C1, R13.1
- removed net N$15: Q2.R2, R14.2
- removed net N$4: D1.C, R5.1
- removed net N$6: D3.C, R3.1
- removed net PG: R5.2, U3.!PG
- removed net STAT1: R3.2, U3.STAT1
- removed net STAT2: R4.2, U3.STAT2
- new net N$12: P1.S, R6.1, U3.IN+
- net +3V3: now also R6.2, U3.V+; no longer R8.2, U1.V+
- net +5V: now also U1.VIN; no longer D1.A, D3.A, Q2.ON/OFF, U3.VDD
- net GND: now also P1.A, R4.1, R5.1, U1.GND, U3.V-; no longer R10.1, R14.1, R6.1, R7.1, U1.V-, U3.VSS
- net N$1: now also R3.2, U1.!CHG; no longer R8.1, R9.2
- net N$10: now also R8.1; no longer R11.1
- net N$2: now also C5.1, R7.2, U3.IN-; no longer C7.1, R12.2, U1.IN-
- net N$3: now also D1.C; no longer LED1.2
- net N$5: now also R3.1; no longer R4.1
- net N$7: now also R7.1, R9.2; no longer R10.2, R12.1
- net N$8: now also C5.2, R8.2, U3.OUT; no longer C7.2, R11.2, U1.OUT
- net PROG: now also R4.2, U1.ISET; no longer R6.2, U3.PROG
- net THERM: now also R5.2, U1.TS; no longer R7.2, U3.THERM
- net V_BATT: now also C2.1, D1.A, U1.OUT; no longer C5.1, LED1.1, Q2.VOUT/C1@1, Q2.VOUT/C1@2
Other:
- note added: "1M"
- note removed: "TODO draw LED PCB add thumbpot"
- moved on the sheet: C2, C5, D1, D2, H1, H2, J1, R3, R4, R5, R6, R7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
